File: Electronics/out/AtlasPower4S/AtlasPower4S.kicad_sch (KiCad schematic)
At the start: 84 parts, among them J1 XT90 / 4S LiPo in, J2 E-STOP, J3 I2C / Qwiic, J4 Jetson 10V, J5 TiM561 10V, J6 servo 7.4V, J7 PPM in, J8 5V out, Q1 ASS053N06Q1M-R, U1 LM74700QDBVRQ1, U2 INA226AIDGSR, U3 AP64501SP-13, U4 AP64501SP-13, U5 AP64501SP-13

Commit message: Electronics: lay out the AtlasPower-4S board, and a real SRP1265A footprint
The two things flagged as unverified last time.

Inductor land pattern: KiCad ships none for the SRP1265A, so gen_footprint.py builds it
from the datasheet Recommended Layout (14.2 mm span, 8.0 gap, 5.0 pad height -> 3.1 x 5.0
pads at +-5.55). Read off the rendered drawing rather than extracted text. It checks out:
3.1 x 5.0 is exactly the worst-case terminal, which is what a power-inductor land is.

Layout: 4 layers, 88 x 68, M3 on 76 x 56 to match the printed tray. layout.py is the hand
floorplan; relax.py separates it numerically until no courtyard overlaps and nothing hangs
off the edge, which the hand coordinates did in six places. Power is zones, signals are
routed with collision checking, and a connection that cannot be routed cleanly is left
unrouted and reported rather than shorted.

DRC 659 -> 204, fixing 54 courtyard overlaps, 90 routing shorts, 47 dangling vias, unfilled
zones, the INA226 exposed pad left unmapped, and footprints whose built-in thermal vias are
under the minimum hole size. The remainder is a GUI cleanup pass and the README says so;
do not order until it is done.
Parts:
- L1, L2, L3: footprint Inductor_SMD:L_APV_APH1265 -> atlaspower:L_Bourns_SRP1265A
- U2: footprint Package_SO:MSOP-10-1EP_3x3mm_P0.5mm_EP1.68x1.88mm_ThermalVias -> Package_SO:MSOP-10-1EP_3x3mm_P0.5mm_EP1.68x1.88mm
- U3, U4, U5: footprint Package_SO:SOIC-8-1EP_3.9x4.9mm_P1.27mm_EP2.29x3mm_ThermalVias -> Package_SO:SOIC-8-1EP_3.9x4.9mm_P1.27mm_EP2.29x3mm
Changed lines of the file:
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@@
     (property "Reference" "U2" (at 116.84 53.88 0) (effects (font (size 1.27 1.27))))
     (property "Value" "INA226AIDGSR" (at 116.84 73.12 0) (effects (font (size 1.27 1.27))))
-    (property "Footprint" "Package_SO:MSOP-10-1EP_3x3mm_P0.5mm_EP1.68x1.88mm_ThermalVias" (at 116.84 63.50 0) (effects (font (size 1.27 1.27)) (hide yes)))
+    (property "Footprint" "Package_SO:MSOP-10-1EP_3x3mm_P0.5mm_EP1.68x1.88mm" (at 116.84 63.50 0) (effects (font (size 1.27 1.27)) (hide yes)))
     (property "LCSC" "C49851" (at 116.84 63.50 0) (effects (font (size 1.27 1.27)) (hide yes)))
     (property "MPN" "INA226AIDGSR" (at 116.84 63.50 0) (effects (font (size 1.27 1.27)) (hide yes)))
@@
     (property "Reference" "U3" (at 332.74 53.88 0) (effects (font (size 1.27 1.27))))
     (property "Value" "AP64501SP-13" (at 332.74 73.12 0) (effects (font (size 1.27 1.27))))
-    (property "Footprint" "Package_SO:SOIC-8-1EP_3.9x4.9mm_P1.27mm_EP2.29x3mm_ThermalVias" (at 332.74 63.50 0) (effects (font (size 1.27 1.27)) (hide yes)))
+    (property "Footprint" "Package_SO:SOIC-8-1EP_3.9x4.9mm_P1.27mm_EP2.29x3mm" (at 332.74 63.50 0) (effects (font (size 1.27 1.27)) (hide yes)))
     (property "LCSC" "C2071517" (at 332.74 63.50 0) (effects (font (size 1.27 1.27)) (hide yes)))
     (property "MPN" "AP64501SP-13" (at 332.74 63.50 0) (effects (font (size 1.27 1.27)) (hide yes)))
@@
     (property "Reference" "L1" (at 30.48 91.98 0) (effects (font (size 1.27 1.27))))
     (property "Value" "10uH/15.5A" (at 30.48 101.06 0) (effects (font (size 1.27 1.27))))
-    (property "Footprint" "Inductor_SMD:L_APV_APH1265" (at 30.48 96.52 0) (effects (font (size 1.27 1.27)) (hide yes)))
+    (property "Footprint" "atlaspower:L_Bourns_SRP1265A" (at 30.48 96.52 0) (effects (font (size 1.27 1.27)) (hide yes)))
     (property "LCSC" "C840531" (at 30.48 96.52 0) (effects (font (size 1.27 1.27)) (hide yes)))
     (property "MPN" "SRP1265A-100M" (at 30.48 96.52 0) (effects (font (size 1.27 1.27)) (hide yes)))
@@
     (property "Reference" "U4" (at 116.84 152.94 0) (effects (font (size 1.27 1.27))))
     (property "Value" "AP64501SP-13" (at 116.84 172.18 0) (effects (font (size 1.27 1.27))))
-    (property "Footprint" "Package_SO:SOIC-8-1EP_3.9x4.9mm_P1.27mm_EP2.29x3mm_ThermalVias" (at 116.84 162.56 0) (effects (font (size 1.27 1.27)) (hide yes)))
+    (property "Footprint" "Package_SO:SOIC-8-1EP_3.9x4.9mm_P1.27mm_EP2.29x3mm" (at 116.84 162.56 0) (effects (font (size 1.27 1.27)) (hide yes)))
     (property "LCSC" "C2071517" (at 116.84 162.56 0) (effects (font (size 1.27 1.27)) (hide yes)))
     (property "MPN" "AP64501SP-13" (at 116.84 162.56 0) (effects (font (size 1.27 1.27)) (hide yes)))
@@
     (property "Reference" "L2" (at 160.02 158.02 0) (effects (font (size 1.27 1.27))))
     (property "Value" "10uH/15.5A" (at 160.02 167.10 0) (effects (font (size 1.27 1.27))))
-    (property "Footprint" "Inductor_SMD:L_APV_APH1265" (at 160.02 162.56 0) (effects (font (size 1.27 1.27)) (hide yes)))
+    (property "Footprint" "atlaspower:L_Bourns_SRP1265A" (at 160.02 162.56 0) (effects (font (size 1.27 1.27)) (hide yes)))
     (property "LCSC" "C840531" (at 160.02 162.56 0) (effects (font (size 1.27 1.27)) (hide yes)))
     (property "MPN" "SRP1265A-100M" (at 160.02 162.56 0) (effects (font (size 1.27 1.27)) (hide yes)))
@@
     (property "Reference" "U5" (at 246.38 218.98 0) (effects (font (size 1.27 1.27))))
     (property "Value" "AP64501SP-13" (at 246.38 238.22 0) (effects (font (size 1.27 1.27))))
-    (property "Footprint" "Package_SO:SOIC-8-1EP_3.9x4.9mm_P1.27mm_EP2.29x3mm_ThermalVias" (at 246.38 228.60 0) (effects (font (size 1.27 1.27)) (hide yes)))
+    (property "Footprint" "Package_SO:SOIC-8-1EP_3.9x4.9mm_P1.27mm_EP2.29x3mm" (at 246.38 228.60 0) (effects (font (size 1.27 1.27)) (hide yes)))
     (property "LCSC" "C2071517" (at 246.38 228.60 0) (effects (font (size 1.27 1.27)) (hide yes)))
     (property "MPN" "AP64501SP-13" (at 246.38 228.60 0) (effects (font (size 1.27 1.27)) (hide yes)))
@@
     (property "Reference" "L3" (at 289.56 224.06 0) (effects (font (size 1.27 1.27))))
     (property "Value" "10uH/15.5A" (at 289.56 233.14 0) (effects (font (size 1.27 1.27))))
-    (property "Footprint" "Inductor_SMD:L_APV_APH1265" (at 289.56 228.60 0) (effects (font (size 1.27 1.27)) (hide yes)))
+    (property "Footprint" "atlaspower:L_Bourns_SRP1265A" (at 289.56 228.60 0) (effects (font (size 1.27 1.27)) (hide yes)))
     (property "LCSC" "C840531" (at 289.56 228.60 0) (effects (font (size 1.27 1.27)) (hide yes)))
     (property "MPN" "SRP1265A-100M" (at 289.56 228.60 0) (effects (font (size 1.27 1.27)) (hide yes)))
